Commit message: After aruco detection

File: dew_ws/src/mini_robot/description/robot.urdf.xacro (robot description, xacro)
@@ -1,14 +1,7 @@
 <?xml version="1.0"?>
 <robot xmlns:xacro="http://www.ros.org/wiki/xacro"  name="robot">
-    <xacro:arg name="use_ros2_control" default="true"/>
     <xacro:arg name="sim_mode" default="false"/>
     <xacro:include filename="robot_core.xacro" />
-    <xacro:if value="$(arg use_ros2_control)">
-        <xacro:include filename="ros2_control.xacro" />
-    </xacro:if>
-    <xacro:unless value="$(arg use_ros2_control)">
-        <xacro:include filename="gazebo_control.xacro" />
-    </xacro:unless>
-    <!-- <xacro:include filename="lidar.xacro" /> -->
     <xacro:include filename="camera.xacro" />
+    <xacro:include filename="gazebo_control.xacro" />
 </robot>

File: dew_ws/src/mini_robot/description/robot_core.xacro (robot description, xacro)
@@ -16,18 +16,4 @@
     <xacro:property name="caster_wheel_offset_x" value="0.07"/>
     <xacro:property name="caster_wheel_offset_z" value="${wheel_offset_z - wheel_radius + caster_wheel_radius}"/>
-     <!-- <xacro:property name="chassis_length" value="0.335"/>
-     <xacro:property name="chassis_width" value="0.265"/>
-     <xacro:property name="chassis_height" value="0.138"/>
-     <xacro:property name="chassis_mass" value="1.0"/>
-     <xacro:property name="wheel_radius" value="0.033"/>
-     <xacro:property name="wheel_thickness" value="0.026"/>
-     <xacro:property name="wheel_mass" value="0.05"/>
-     <xacro:property name="wheel_offset_x" value="0.226"/>
-     <xacro:property name="wheel_offset_y" value="0.1485"/>
-     <xacro:property name="wheel_offset_z" value="0.01"/>
-     <xacro:property name="caster_wheel_radius" value="0.01"/>
-     <xacro:property name="caster_wheel_mass" value="0.01"/>
-     <xacro:property name="caster_wheel_offset_x" value="0.075"/>
-     <xacro:property name="caster_wheel_offset_z" value="${wheel_offset_z - wheel_radius + caster_wheel_radius}"/> -->
     <material name="white">
         <color rgba="1 1 1 1" />
